File: wifi-board.sch (EAGLE design)
At the start: 21 parts

Commit message: updated battery connector
Parts:
- added LOGO2: ROBOKODING-LOGOM, Sumorobot:ROBOKODING-LOGOM
- added POWER: SPDT_SLIDE_SWITCH, custom:SPDT_SLIDE_SWITCH
- renumbered LEFT_LINE to L-LINE, LEFT_SERVO to L-SERVO, RIGHT_LINE to R-LINE, RIGHT_SERVO to R-SERVO
Connections:
- new net BAT_IN: BATTERY.2, POWER.COMMON
- net RST: no longer ARDUINO.RST
- net VIN: now also POWER.SW2; no longer BATTERY.2
Other:
- note added: "Power input and conversion"
- note removed: "Battery & Power converter"
- moved on the sheet: BATTERY, CONVERTER

Commit message: updated power connector and resistors
Parts:
- BATTERY: value M02JST-PTH-VERT -> M02LOCK_LONGPADS; device SparkFun-Connectors:M02JST-PTH-VERT -> SparkFun-Connectors:M02LOCK_LONGPADS
- LOGO2: device Sumorobot:ROBOKODING-LOGOM -> robokoding-logo:ROBOKODING-LOGOM
- R5, R7: value 10K -> 4K7
- renumbered ARDUINO to MCU, WIFI_MODULE to COM_MODULE
Connections:
- net +3V3: now also R5.1, R7.1
- net GND: no longer R5.1, R7.1
Other:
- note added: "Communication module"
- note added: "Microcontroller"
- note added: "Microcontroller auto reset"
- note removed: "Arduino Pro Mini"
- note removed: "Max Current Output: 1000mA"
- note removed: "USR-WIFI-T module"
- note removed: "Voltage Input: 1.5~5.5VDC"
- note removed: "Voltage Output: 5VDC"
- note removed: "WIFI Arduino reset"
- moved on the sheet: CONVERTER
